File: aom-preamp.kicad_pcb (KiCad board)
At the start: 2 copper layers, 81 x 26.5 mm, 47 parts, among them J1 Battery_9V, J3 USB_B_Mini, J4 PJ-320B, Q1 BC849, Q2 BC859, Q3 BC859, Q4 BC859, Q5 BC849, U1 CM108B, U2 PC817

Commit message: update
Parts:
- removed JP3: PullUp, Jumper:SolderJumper-2_P1.3mm_Open_RoundedPad1.0x1.5mm
- removed R11: 10R, Resistor_SMD:R_0805_2012Metric
- added M1: MountingHole_2.7mm_M2.5, MountingHole:MountingHole_2.7mm_M2.5, F.Cu at (95.5, 79.0)
- added M2: MountingHole_2.7mm_M2.5, MountingHole:MountingHole_2.7mm_M2.5, F.Cu at (95.5, 99.0)
- added M3: MountingHole_2.7mm_M2.5, MountingHole:MountingHole_2.7mm_M2.5, F.Cu at (168.5, 99.0)
- added M4: MountingHole_2.7mm_M2.5, MountingHole:MountingHole_2.7mm_M2.5, F.Cu at (168.5, 79.0)
- moved J1 26.8 mm to (153.1, 80.2)
- moved U2 23.0 mm to (135.3, 80.3)
- moved R17 19.7 mm to (132.0, 85.4)
- moved C7 14.5 mm to (132.5, 93.0)
- moved R14 12.9 mm to (158.0, 95.4)
- moved R8 11.6 mm to (135.4, 99.5)
- moved Q5 10.7 mm to (136.1, 86.1), turned to 90 degrees
- moved FB2 10.7 mm to (156.3, 86.5)
- moved C4 10.2 mm to (130.4, 98.0)
- moved R16 7.94 mm to (143.0, 81.6), turned to -90 degrees
- moved R15 7.05 mm to (160.4, 77.5), turned to 180 degrees
- moved D1 5.59 mm to (160.2, 82.0), turned to 180 degrees
- moved C14 5.35 mm to (156.5, 99.5), turned to -90 degrees
- moved R12 5.23 mm to (160.0, 91.4), turned to 90 degrees
- moved R5 4.30 mm to (126.5, 94.6), turned to 90 degrees
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Connections:
- C2 pad 2: GND1 -> GND
- C3 pad 2: GND1 -> GND
- C5 pad 1: Net-(Q4-E) -> 9V_BAT
- C5 pad 2: GND1 -> GND
- C6 pad 1: GND1 -> GND
- C6 pad 2: Net-(Q4-E) -> 9V_BAT
- C7 pad 2: GND1 -> GND
- J4 pad 2: GND1 -> GND
- Q1 pad 2: GND1 -> GND
- Q4 pad 2: Net-(Q4-E) -> 9V_BAT
- Q5 pad 3: GND1 -> GND
- R10 pad 1: Net-(Q4-E) -> 9V_BAT
- R2 pad 2: GND1 -> GND
- R3 pad 1: Net-(Q4-E) -> 9V_BAT
- R4 pad 1: Net-(Q4-E) -> 9V_BAT
- R7 pad 1: GND1 -> GND
- R9 pad 2: GND1 -> GND
Routing:
- net GND: track 0.00 -> 163.5 mm, vias 0 -> 11
- net V3.3: track 0.00 -> 39.4 mm, vias 0 -> 4
- net Net-(J3-Shield): track 0.00 -> 28.1 mm
- net AVDD1: track 0.00 -> 27.9 mm
- net 9V_GND: track 0.00 -> 21.5 mm
- net Net-(Q1-C): track 0.00 -> 21.3 mm
- net Net-(Q2-E): track 0.00 -> 20.5 mm, vias 0 -> 2
- net Net-(C2-Pad1): track 0.00 -> 20.2 mm
- net Net-(C1-Pad1): track 0.00 -> 19.9 mm
- net LEDO: track 0.00 -> 17.9 mm
- net Net-(Q1-B): track 0.00 -> 17.7 mm, vias 0 -> 4
- net Net-(R16-Pad1): track 0.00 -> 16.0 mm, vias 0 -> 2
- net Net-(Q3-B): track 0.00 -> 13.6 mm, vias 0 -> 2
- net Net-(R12-Pad1): track 0.00 -> 13.3 mm, vias 0 -> 2
- net Net-(R13-Pad1): track 0.00 -> 11.7 mm
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- added copper zone on F.Cu, net 9V_BAT
- added copper zone on B.Cu, net GND
- added copper zone on F.Cu, net V3.3
Other:
- board size 81 x 26.5 mm -> 80 x 27 mm

Commit message: update
Parts:
- moved FB2 13.2 mm to (164.5, 96.8), turned to 90 degrees
- moved R15 9.51 mm to (160.0, 87.0)
- moved R17 9.00 mm to (141.0, 85.6)
- moved R7 5.12 mm to (122.6, 87.5)
- moved R16 4.55 mm to (147.0, 79.4)
- moved JP2 4.09 mm to (157.5, 91.3), turned to -90 degrees
- moved F2 3.78 mm to (142.5, 79.8), turned to -90 degrees
- moved Q1 3.68 mm to (122.0, 91.5)
- moved R13 3.00 mm to (154.5, 91.4)
- moved D1 2.69 mm to (161.2, 79.5), turned to 0 degrees
- moved F1 2.00 mm to (161.5, 99.0), turned to -90 degrees
- moved C13 1.50 mm to (151.5, 99.5), turned to -90 degrees
- moved J1 1.25 mm to (153.1, 81.5)
- moved C12 1.12 mm to (141.5, 98.5)
- moved C11 1.10 mm to (148.0, 99.5), turned to -90 degrees
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Connections:
- F1 pad 1: AVDD1 -> Net-(F1-Pad1)
- F1 pad 2: VBUS -> AVDD1
- FB1 pad 2: VBUS -> Net-(F1-Pad1)
- U1 pad 35: VDD -> AVDD1
Routing:
- net GND: track 163.5 -> 39.8 mm, vias 11 -> 6
- net 9V_BAT: track 6.93 -> 52.6 mm
- net 9V_GND: track 21.5 -> 7.74 mm, vias 0 -> 4
- net Net-(Q3-E): track 3.46 -> 15.0 mm, vias 0 -> 2
- net Net-(J3-Shield): track 28.1 -> 22.4 mm
- net LEDO: track 17.9 -> 12.4 mm
- net Net-(JP2-B): track 7.85 -> 2.71 mm
- net Net-(J1-Pin_1): track 6.24 -> 10.7 mm
- net Net-(R17-Pad2): track 8.38 -> 4.43 mm
- net V3.3: track 39.4 -> 43.1 mm, vias 4 -> 2
- net Net-(Q3-B): track 13.6 -> 16.6 mm
- net VBUS: track 3.04 -> 0.00 mm
- net AVDD1: track 27.9 -> 30.9 mm, vias 0 -> 2
- net Net-(C3-Pad1): track 8.25 -> 5.39 mm
- net Net-(Q1-B): track 17.7 -> 15.0 mm, vias 4 -> 2
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- added copper zone on B.Cu, net 9V_GND
- added copper zone on F.Cu, net GND
- removed copper zone on F.Cu, net 9V_BAT
- removed copper zone on B.Cu, net GND
- removed copper zone on F.Cu, net V3.3
Other:
- board text added: "+9V"
- board text added: "GND"

Commit message: Update project files
Parts:
- C1, C2, C3, C5: footprint Capacitor_SMD:CP_Elec_6.3x7.7 -> Capacitor_SMD:CP_Elec_5x5.4
- C4: value 100uF -> +100uF; footprint Capacitor_SMD:C_0805_2012Metric -> Capacitor_SMD:CP_Elec_5x5.4
- FB1: value 160R@ 100MhZ -> 30mOhm
- FB2: value 160R @ 100Mhz -> 30mOhm
- moved R5 5.00 mm to (121.5, 97.4)
- moved C3 3.18 mm to (115.3, 98.0)
- moved R6 2.00 mm to (124.5, 97.4), turned to 90 degrees
- moved C4 1.51 mm to (130.3, 99.5)
- moved R8 1.18 mm to (136.6, 99.5)
- moved C2 1.13 mm to (107.2, 98.0)
- moved C5 0.90 mm to (108.7, 79.5)
- moved C7 0.71 mm to (133.0, 92.5)
- moved C1 0.69 mm to (108.5, 88.5)
Routing:
- net Net-(Q2-E): track 21.9 -> 18.9 mm
- net Net-(Q1-C): track 19.3 -> 18.0 mm
- net Net-(C3-Pad1): track 5.39 -> 4.53 mm
- net 9V_BAT: track 52.6 -> 51.9 mm
- net Net-(C4-Pad2): track 3.72 -> 3.18 mm
Other:
- board text added: "9V Battery to power preamp"
- board text added: "Electret Capsule Microphone"
- board text added: "JLCJLC"
- board text added: "LED_OP"
- board text added: "USB MINI Output"
