File: aom-preamp.kicad_sch (KiCad schematic)
At the start: 46 parts, among them J1 Battery_9V, J2 AudioJack3, J3 USB_B_Mini, Q1 BC849, Q2 BC859, Q3 BC859, Q4 BC859, Q5 BC849, U1 CM108B, U2 PC817

Commit message: Update project files
Parts:
- removed J2: AudioJack3, Connector_Audio:Jack_3.5mm_PJ311_Horizontal, symbol Connector_Audio:AudioJack3
- added J4: PJ-320B, BOOMELE_PJ-320B:BOOMELE_PJ-320B, symbol PJ-320B:PJ-320B
- added JP3: PullUp, Jumper:SolderJumper-2_P1.3mm_Open_RoundedPad1.0x1.5mm, symbol Jumper:SolderJumper_2_Open
- J1: footprint Connector_PinHeader_2.54mm:PinHeader_1x02_P2.54mm_Vertical -> Connector_JST:JST_PH_B2B-PH-SM4-TB_1x02-1MP_P2.00mm_Vertical
- JP2: footprint Jumper:SolderJumper-3_P1.3mm_Open_Pad1.0x1.5mm -> Jumper:SolderJumper-2_P1.3mm_Open_RoundedPad1.0x1.5mm
Connections:
- net GND: now also JP3.2 (B); no longer C2.2, C3.2, C5.2, C6.1, C7.2, Q1.2 (E), Q5.3 (C), R2.2, R7.1, R9.2
- net at C1.1, R3.2: now also J4.3
- new net GND1: C2.2, C3.2, C5.2, C6.1, C7.2, J4.2, JP3.1 (A), Q1.2 (E), Q5.3 (C), R2.2, R7.1, R9.2
Other:
- note added: "AUDIO OUT GND"
- note removed: "SAME GND"

Commit message: update
Parts:
- removed JP3: PullUp, Jumper:SolderJumper-2_P1.3mm_Open_RoundedPad1.0x1.5mm, symbol Jumper:SolderJumper_2_Open
- removed R11: 10R, Resistor_SMD:R_0805_2012Metric, symbol Device:R
Connections:
- net GND1 is gone; now on net GND: C2.2, C3.2, C5.2, C6.1, C7.2, J4.2, Q1.2 (E), Q5.3 (C), R2.2, R7.1, R9.2
- net 9V_BAT: now also C5.1, C6.2, Q4.2 (E), R10.1, R3.1, R4.1
Other:
- note removed: "AUDIO OUT GND"

Commit message: update
Connections:
- net VDD is gone; now on net AVDD1: U1.35
- net AVDD1: now also F1.2; no longer F1.1
- net VBUS: no longer names the net of FB1.2
- net VBUS: now also F1.1; no longer F1.2
Other:
- moved on the sheet: F1
Changed lines of the file:
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@@
-	(wire
-		(pts
-			(xy 166.37 53.34) (xy 171.45 53.34)
-		)
-		(stroke
-			(width 0)
-			(type default)
-		)
-	)
 	(wire
 		(pts
@@
 		)
 	)
+	(global_label "VDD"
+		(shape input)
+		(at 158.75 53.34 0)
+		(fields_autoplaced yes)
+		(effects
+			(font
+				(size 1.27 1.27)
+			)
+			(justify left)
+		)
+		(property "Intersheetrefs" "${INTERSHEET_REFS}"
+			(at 165.3638 53.34 0)
+			(effects
+				(font
+					(size 1.27 1.27)
+				)
+				(justify left)
+				(hide yes)
+			)
+		)
+	)
 	(global_label "DM"
 		(shape input)
@@
 		)
 	)
-	(global_label "VBUS"
+	(global_label "9V_BAT"
 		(shape input)
-		(at 171.45 53.34 0)
+		(at 129.54 29.21 90)
 		(fields_autoplaced yes)
 		(effects
@@
 		)
 		(property "Intersheetrefs" "${INTERSHEET_REFS}"
-			(at 179.3338 53.34 0)
-			(effects
-				(font
-					(size 1.27 1.27)
-				)
-				(justify left)
-				(hide yes)
-			)
-		)
-	)
-	(global_label "9V_BAT"
+			(at 129.54 19.6329 90)
+			(effects
+				(font
+					(size 1.27 1.27)
+				)
+				(justify left)
+				(hide yes)
+			)
+		)
+	)
+	(global_label "V3.3"
 		(shape input)
-		(at 129.54 29.21 90)
+		(at 236.22 30.48 90)
 		(fields_autoplaced yes)
 		(effects
@@
 		)
 		(property "Intersheetrefs" "${INTERSHEET_REFS}"
-			(at 129.54 19.6329 90)
-			(effects
-				(font
-					(size 1.27 1.27)
-				)
-				(justify left)
-				(hide yes)
-			)
-		)
-	)
-	(global_label "V3.3"
+			(at 236.22 23.3824 90)
+			(effects
+				(font
+					(size 1.27 1.27)
+				)
+				(justify left)
+				(hide yes)
+			)
+		)
+	)
+	(global_label "LEDO"
 		(shape input)
-		(at 236.22 30.48 90)
+		(at 207.01 85.09 180)
 		(fields_autoplaced yes)
 		(effects
@@
 				(size 1.27 1.27)
 			)
-			(justify left)
+			(justify right)
 		)
 		(property "Intersheetrefs" "${INTERSHEET_REFS}"
-			(at 236.22 23.3824 90)
-			(effects
-				(font
-					(size 1.27 1.27)
-				)
-				(justify left)
-				(hide yes)
-			)
-		)
-	)
-	(global_label "LEDO"
+			(at 199.2472 85.09 0)
+			(effects
+				(font
+					(size 1.27 1.27)
+				)
+				(justify right)
+				(hide yes)
+			)
+		)
+	)
+	(global_label "MIC_IN"
 		(shape input)
-		(at 207.01 85.09 180)
+		(at 255.27 80.01 0)
 		(fields_autoplaced yes)
 		(effects
@@
 				(size 1.27 1.27)
 			)
-			(justify right)
+			(justify left)
 		)
 		(property "Intersheetrefs" "${INTERSHEET_REFS}"
-			(at 199.2472 85.09 0)
-			(effects
-				(font
-					(size 1.27 1.27)
-				)
-				(justify right)
-				(hide yes)
-			)
-		)
-	)
-	(global_label "MIC_IN"
+			(at 264.4843 80.01 0)
+			(effects
+				(font
+					(size 1.27 1.27)
+				)
+				(justify left)
+				(hide yes)
+			)
+		)
+	)
+	(global_label "AVDD1"
 		(shape input)
-		(at 255.27 80.01 0)
+		(at 177.8 77.47 0)
 		(fields_autoplaced yes)
 		(effects
@@
 		)
 		(property "Intersheetrefs" "${INTERSHEET_REFS}"
-			(at 264.4843 80.01 0)
-			(effects
-				(font
-					(size 1.27 1.27)
-				)
-				(justify left)
-				(hide yes)
-			)
-		)
-	)
-	(global_label "AVDD1"
+			(at 186.7119 77.47 0)
+			(effects
+				(font
+					(size 1.27 1.27)
+				)
+				(justify left)
+				(hide yes)
+			)
+		)
+	)
+	(global_label "9V_GND"
 		(shape input)
-		(at 177.8 77.47 0)
+		(at 228.6 157.48 180)
 		(fields_autoplaced yes)
 		(effects
@@
 				(size 1.27 1.27)
 			)
-			(justify left)
+			(justify right)
 		)
 		(property "Intersheetrefs" "${INTERSHEET_REFS}"
-			(at 186.7119 77.47 0)
-			(effects
-				(font
-					(size 1.27 1.27)
-				)
-				(justify left)
-				(hide yes)
-			)
-		)
-	)
-	(global_label "9V_GND"
+			(at 218.4786 157.48 0)
+			(effects
+				(font
+					(size 1.27 1.27)
+				)
+				(justify right)
+				(hide yes)
+			)
+		)
+	)
+	(global_label "9V_BAT"
 		(shape input)
-		(at 228.6 157.48 180)
+		(at 252.73 125.73 90)
 		(fields_autoplaced yes)
 		(effects
@@
 				(size 1.27 1.27)
 			)
-			(justify right)
+			(justify left)
 		)
 		(property "Intersheetrefs" "${INTERSHEET_REFS}"
-			(at 218.4786 157.48 0)
-			(effects
-				(font
-					(size 1.27 1.27)
-				)
-				(justify right)
-				(hide yes)
-			)
-		)
-	)
-	(global_label "VBUS"
+			(at 252.73 116.1529 90)
+			(effects
+				(font
+					(size 1.27 1.27)
+				)
+				(justify left)
+				(hide yes)
+			)
+		)
+	)
+	(global_label "AVDD1"
 		(shape input)
-		(at 177.8 130.81 0)
+		(at 256.54 74.93 0)
 		(fields_autoplaced yes)
 		(effects
@@
 		)
 		(property "Intersheetrefs" "${INTERSHEET_REFS}"
-			(at 185.6838 130.81 0)
-			(effects
-				(font
-					(size 1.27 1.27)
-				)
-				(justify left)
-				(hide yes)
-			)
-		)
-	)
-	(global_label "9V_BAT"
+			(at 265.4519 74.93 0)
+			(effects
+				(font
+					(size 1.27 1.27)
+				)
+				(justify left)
+				(hide yes)
+			)
+		)
+	)
+	(global_label "VDD"
 		(shape input)
-		(at 252.73 125.73 90)
+		(at 185.42 130.81 0)
 		(fields_autoplaced yes)
 		(effects
@@
 		)
 		(property "Intersheetrefs" "${INTERSHEET_REFS}"
-			(at 252.73 116.1529 90)
-			(effects
-				(font
-					(size 1.27 1.27)
-				)
-				(justify left)
-				(hide yes)
-			)
-		)
-	)
-	(global_label "AVDD1"
-		(shape input)
-		(at 256.54 74.93 0)
-		(fields_autoplaced yes)
-		(effects
-			(font
-				(size 1.27 1.27)
-			)
-			(justify left)
-		)
-		(property "Intersheetrefs" "${INTERSHEET_REFS}"
-			(at 265.4519 74.93 0)
+			(at 192.0338 130.81 0)
 			(effects
 				(font
@@
 	(symbol
 		(lib_id "Device:Polyfuse")
-		(at 162.56 53.34 90)
+		(at 181.61 130.81 90)
 		(unit 1)
 		(exclude_from_sim no)
@@
 		(on_board yes)
 		(dnp no)
-		(fields_autoplaced yes)
 		(property "Reference" "F1"
-			(at 162.56 46.99 90)
+			(at 183.896 135.128 90)
 			(effects
 				(font
@@
 		)
 		(property "Value" "MF-FSMF050X-2"
-			(at 162.56 49.53 90)
+			(at 182.372 133.096 90)
 			(effects
 				(font
@@
 		)
 		(property "Footprint" "Fuse:Fuse_0603_1608Metric"
-			(at 167.64 52.07 0)
+			(at 186.69 129.54 0)
 			(effects
 				(font
@@
 		)
 		(property "Datasheet" "~"
-			(at 162.56 53.34 0)
+			(at 181.61 130.81 0)
 			(effects
 				(font
@@
 		)
 		(property "Description" "Resettable fuse, polymeric positive temperature coefficient"
-			(at 162.56 53.34 0)
-			(effects
-				(font
+			(at 181.61 130.81 0)
+			(effects
+				(font

Commit message: Update project files
Parts:
- C1, C2, C3, C5: footprint Capacitor_SMD:CP_Elec_6.3x7.7 -> Capacitor_SMD:CP_Elec_5x5.4
- C4: value 100uF -> +100uF; footprint Capacitor_SMD:C_0805_2012Metric -> Capacitor_SMD:CP_Elec_5x5.4
- FB1: value 160R@ 100MhZ -> 30mOhm
- FB2: value 160R @ 100Mhz -> 30mOhm
Other:
- moved on the sheet: F1
Changed lines of the file:
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@@
 	(wire
 		(pts
+			(xy 190.5 130.81) (xy 194.31 130.81)
+		)
+		(stroke
+			(width 0)
+			(type default)
+		)
+	)
+	(wire
+		(pts
 			(xy 158.75 59.69) (xy 168.91 59.69)
 		)
@@
 	(wire
 		(pts
-			(xy 175.26 130.81) (xy 177.8 130.81)
+			(xy 175.26 130.81) (xy 182.88 130.81)
 		)
 		(stroke
@@
 	(global_label "VDD"
 		(shape input)
-		(at 185.42 130.81 0)
+		(at 194.31 130.81 0)
 		(fields_autoplaced yes)
 		(effects
@@
 		)
 		(property "Intersheetrefs" "${INTERSHEET_REFS}"
-			(at 192.0338 130.81 0)
+			(at 200.9238 130.81 0)
 			(effects
 				(font
@@
 			)
 		)
-		(property "Value" "160R@ 100MhZ"
-			(at 177.8 127.508 90)
+		(property "Value" "30mOhm"
+			(at 174.752 127.254 90)
 			(effects
 				(font
@@
 			)
 		)
-		(property "Value" "100uF"
+		(property "Value" "+100uF"
 			(at 109.601 52.07 90)
 			(effects
@@
 			)
 		)
-		(property "Footprint" "Capacitor_SMD:C_0805_2012Metric"
+		(property "Footprint" "Capacitor_SMD:CP_Elec_5x5.4"
 			(at 114.3 56.1848 0)
 			(effects
@@
 			)
 		)
-		(property "Footprint" "Capacitor_SMD:CP_Elec_6.3x7.7"
+		(property "Footprint" "Capacitor_SMD:CP_Elec_5x5.4"
 			(at 68.2752 97.79 0)
 			(effects
@@
 	(symbol
 		(lib_id "Device:Polyfuse")
-		(at 181.61 130.81 90)
+		(at 186.69 130.81 90)
 		(unit 1)
 		(exclude_from_sim no)
@@
 		(dnp no)
 		(property "Reference" "F1"
-			(at 183.896 135.128 90)
+			(at 187.706 128.016 90)
 			(effects
 				(font
@@
 		)
 		(property "Value" "MF-FSMF050X-2"
-			(at 182.372 133.096 90)
+			(at 187.452 133.096 90)
 			(effects
 				(font
@@
 		)
 		(property "Footprint" "Fuse:Fuse_0603_1608Metric"
-			(at 186.69 129.54 0)
+			(at 191.77 129.54 0)
 			(effects
 				(font
@@
 		)
 		(property "Datasheet" "~"
-			(at 181.61 130.81 0)
+			(at 186.69 130.81 0)
 			(effects
 				(font
@@
 		)
 		(property "Description" "Resettable fuse, polymeric positive temperature coefficient"
-			(at 181.61 130.81 0)
+			(at 186.69 130.81 0)
 			(effects
 				(font
@@
 			)
 		)
-		(property "Value" "160R @ 100Mhz"
+		(property "Value" "30mOhm"
 			(at 164.338 148.59 0)
 			(effects
@@
 			)
 		)
-		(property "Datasheet" ""
+		(property "Datasheet" "https://www.lcsc.com/product-detail/Audio-Connectors_SHOU-HAN-PJ-320-3P-SMT_C17701688.html"
 			(at 29.21 68.58 0)
 			(effects
@@
 			)
 		)
-		(property "Description" ""
+		(property "Description" "C17701688"
 			(at 29.21 68.58 0)
 			(effects
@@
 			)
 		)
-		(property "Footprint" "Capacitor_SMD:CP_Elec_6.3x7.7"
+		(property "Footprint" "Capacitor_SMD:CP_Elec_5x5.4"
 			(at 53.34 70.1548 0)
 			(effects
@@
 			)
 		)
-		(property "Footprint" "Capacitor_SMD:CP_Elec_6.3x7.7"
+		(property "Footprint" "Capacitor_SMD:CP_Elec_5x5.4"
 			(at 68.2752 41.91 0)
 			(effects
@@
 			)
 		)
-		(property "Footprint" "Capacitor_SMD:CP_Elec_6.3x7.7"
+		(property "Footprint" "Capacitor_SMD:CP_Elec_5x5.4"
 			(at 58.1152 92.71 0)
 			(effects
